File: pcb/onyks-iot-esp32-storage-rfid/peripherials.kicad_sch (KiCad schematic)
At the start: 2 parts, among them J5 Conn_01x03_Pin, J6 Conn_01x01_Pin

Commit message: oznaczenie pinów i podział elementów PCB
dodanie oznaczenia nieużywanych pinów zgodnie z opinią schematu
Changed lines of the file:
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@@
 (kicad_sch
-	(version 20231120)
+	(version 20250114)
 	(generator "eeschema")
-	(generator_version "8.0")
+	(generator_version "9.0")
 	(paper "A4")
 	(title_block
@@
 		(rev "v1.0")
 		(company "KN ONYKS")
+	)
+	(text_box "External RFID modem connector"
+		(exclude_from_sim no)
+		(at 59.69 27.94 0)
+		(size 33.02 36.83)
+		(margins 0.9525 0.9525 0.9525 0.9525)
+		(stroke
+			(width 0)
+			(type default)
+		)
+		(fill
+			(type none)
+		)
+		(effects
+			(font
+				(size 1.27 1.27)
+			)
+			(justify left top)
+		)
 	)
 	(wire
@@
 		)
 	)
-	(text_box "External RFID modem connector"
-		(exclude_from_sim no)
-		(at 59.69 27.94 0)
-		(size 33.02 36.83)
-		(stroke
-			(width 0)
-			(type default)
-		)
-		(fill
-			(type none)
-		)
-		(effects
-			(font
-				(size 1.27 1.27)
-			)
-			(justify left top)
-		)
-	)

Commit message: projekt PCB v2
Parts:
- removed J5: Conn_01x03_Pin, Connector_PinHeader_2.54mm:PinHeader_1x03_P2.54mm_Vertical, symbol Connector:Conn_01x03_Pin
- removed J6: Conn_01x01_Pin, Connector_PinHeader_2.54mm:PinHeader_1x01_P2.54mm_Vertical, symbol Connector:Conn_01x01_Pin
- added J4: Conn_01x04_Pin, Connector_PinHeader_2.54mm:PinHeader_1x04_P2.54mm_Vertical, symbol Connector:Conn_01x04_Pin
- added R4: 10k, Resistor_SMD:R_0603_1608Metric_Pad0.98x0.95mm_HandSolder, symbol Device:R
Connections:
- net GND: now also J4.4 (Pin_4)
- net RXD: now also J4.3 (Pin_3), R4.1
- net TXD: now also J4.2 (Pin_2)
- net VCC: now also J4.1 (Pin_1), R4.2
Changed lines of the file:
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@@
 	(text_box "External RFID modem connector"
 		(exclude_from_sim no)
-		(at 59.69 27.94 0)
-		(size 33.02 36.83)
+		(at 58.42 26.67 0)
+		(size 52.07 36.83)
 		(margins 0.9525 0.9525 0.9525 0.9525)
 		(stroke
@@
 		)
 	)
+	(junction
+		(at 90.17 52.07)
+		(diameter 0)
+		(color 0 0 0 0)
+	)
+	(wire
+		(pts
+			(xy 90.17 46.99) (xy 90.17 52.07)
+		)
+		(stroke
+			(width 0)
+			(type default)
+		)
+	)
 	(wire
 		(pts
@@
 	(wire
 		(pts
-			(xy 76.2 49.53) (xy 85.09 49.53)
-		)
-		(stroke
-			(width 0)
-			(type default)
-		)
-	)
-	(wire
-		(pts
 			(xy 85.09 54.61) (xy 85.09 55.88)
 		)
@@
 	(wire
 		(pts
-			(xy 76.2 40.64) (xy 85.09 40.64)
-		)
-		(stroke
-			(width 0)
-			(type default)
-		)
-	)
-	(wire
-		(pts
-			(xy 76.2 52.07) (xy 85.09 52.07)
-		)
-		(stroke
-			(width 0)
-			(type default)
-		)
-	)
-	(wire
-		(pts
-			(xy 85.09 39.37) (xy 85.09 40.64)
-		)
-		(stroke
-			(width 0)
-			(type default)
-		)
-	)
-	(hierarchical_label "TXD"
-		(shape output)
-		(at 85.09 52.07 0)
+			(xy 90.17 52.07) (xy 95.25 52.07)
+		)
+		(stroke
+			(width 0)
+			(type default)
+		)
+	)
+	(wire
+		(pts
+			(xy 76.2 46.99) (xy 85.09 46.99)
+		)
+		(stroke
+			(width 0)
+			(type default)
+		)
+	)
+	(wire
+		(pts
+			(xy 76.2 52.07) (xy 90.17 52.07)
+		)
+		(stroke
+			(width 0)
+			(type default)
+		)
+	)
+	(wire
+		(pts
+			(xy 76.2 49.53) (xy 95.25 49.53)
+		)
+		(stroke
+			(width 0)
+			(type default)
+		)
+	)
+	(wire
+		(pts
+			(xy 85.09 39.37) (xy 85.09 46.99)
+		)
+		(stroke
+			(width 0)
+			(type default)
+		)
+	)
+	(hierarchical_label "RXD"
+		(shape input)
+		(at 95.25 52.07 0)
 		(effects
 			(font
@@
 		)
 	)
-	(hierarchical_label "RXD"
-		(shape input)
-		(at 85.09 49.53 0)
+	(hierarchical_label "TXD"
+		(shape output)
+		(at 95.25 49.53 0)
 		(effects
 			(font
@@
 	)
 	(symbol
-		(lib_id "Connector:Conn_01x03_Pin")
-		(at 71.12 52.07 0)
+		(lib_id "Connector:Conn_01x04_Pin")
+		(at 71.12 49.53 0)
 		(unit 1)
 		(exclude_from_sim no)
@@
 		(dnp no)
 		(fields_autoplaced yes)
-		(property "Reference" "J5"
+		(property "Reference" "J4"
+			(at 71.755 41.91 0)
+			(effects
+				(font
+					(size 1.27 1.27)
+				)
+			)
+		)
+		(property "Value" "Conn_01x04_Pin"
 			(at 71.755 44.45 0)
 			(effects
@@
 			)
 		)
-		(property "Value" "Conn_01x03_Pin"
-			(at 71.755 46.99 0)
-			(effects
-				(font
-					(size 1.27 1.27)
-				)
-			)
-		)
-		(property "Footprint" "Connector_PinHeader_2.54mm:PinHeader_1x03_P2.54mm_Vertical"
-			(at 71.12 52.07 0)
+		(property "Footprint" "Connector_PinHeader_2.54mm:PinHeader_1x04_P2.54mm_Vertical"
+			(at 71.12 49.53 0)
 			(effects
 				(font
@@
 		)
 		(property "Datasheet" "~"
-			(at 71.12 52.07 0)
-			(effects
-				(font
-					(size 1.27 1.27)
-				)
-				(hide yes)
-			)
-		)
-		(property "Description" "Generic connector, single row, 01x03, script generated"
-			(at 71.12 52.07 0)
-			(effects
-				(font
-					(size 1.27 1.27)
-				)
-				(hide yes)
-			)
+			(at 71.12 49.53 0)
+			(effects
+				(font
+					(size 1.27 1.27)
+				)
+				(hide yes)
+			)
+		)
+		(property "Description" "Generic connector, single row, 01x04, script generated"
+			(at 71.12 49.53 0)
+			(effects
+				(font
+					(size 1.27 1.27)
+				)
+				(hide yes)
+			)
+		)
+		(pin "3"
 		)
 		(pin "2"
 		)
-		(pin "3"
-		)
 		(pin "1"
+		)
+		(pin "4"
 		)
 		(instances
 			(project ""
 				(path "/d3620cad-99d5-4267-a144-49d6f9957c6b/de20a575-b588-4674-a6be-01e8d6418ae5"
-					(reference "J5")
+					(reference "J4")
 					(unit 1)
 				)
@@
 	)
 	(symbol
-		(lib_id "Connector:Conn_01x01_Pin")
-		(at 71.12 40.64 0)
+		(lib_id "power:VCC")
+		(at 90.17 39.37 0)
 		(unit 1)
 		(exclude_from_sim no)
@@
 		(dnp no)
 		(fields_autoplaced yes)
-		(property "Reference" "J6"
-			(at 71.755 35.56 0)
-			(effects
-				(font
-					(size 1.27 1.27)
-				)
-			)
-		)
-		(property "Value" "Conn_01x01_Pin"
-			(at 71.755 38.1 0)
-			(effects
-				(font
-					(size 1.27 1.27)
-				)
-			)
-		)
-		(property "Footprint" "Connector_PinHeader_2.54mm:PinHeader_1x01_P2.54mm_Vertical"
-			(at 71.12 40.64 0)
+		(property "Reference" "#PWR024"
+			(at 90.17 43.18 0)
+			(effects
+				(font
+					(size 1.27 1.27)
+				)
+				(hide yes)
+			)
+		)
+		(property "Value" "VCC"
+			(at 90.17 34.29 0)
+			(effects
+				(font
+					(size 1.27 1.27)
+				)
+			)
+		)
+		(property "Footprint" ""
+			(at 90.17 39.37 0)
+			(effects
+				(font
+					(size 1.27 1.27)
+				)
+				(hide yes)
+			)
+		)
+		(property "Datasheet" ""
+			(at 90.17 39.37 0)
+			(effects
+				(font
+					(size 1.27 1.27)
+				)
+				(hide yes)
+			)
+		)
+		(property "Description" "Power symbol creates a global label with name \"VCC\""
+			(at 90.17 39.37 0)
+			(effects
+				(font
+					(size 1.27 1.27)
+				)
+				(hide yes)
+			)
+		)
+		(pin "1"
+		)
+		(instances
+			(project "onyks-iot-esp32-storage-rfid"
+				(path "/d3620cad-99d5-4267-a144-49d6f9957c6b/de20a575-b588-4674-a6be-01e8d6418ae5"
+					(reference "#PWR024")
+					(unit 1)
+				)
+			)
+		)
+	)
+	(symbol
+		(lib_id "Device:R")
+		(at 90.17 43.18 180)
+		(unit 1)
+		(exclude_from_sim no)
+		(in_bom yes)
+		(on_board yes)
+		(dnp no)
+		(fields_autoplaced yes)
+		(property "Reference" "R4"
+			(at 92.71 41.9099 0)
+			(effects
+				(font
+					(size 1.27 1.27)
+				)
+				(justify right)
+			)
+		)
+		(property "Value" "10k"
+			(at 92.71 44.4499 0)
+			(effects
+				(font
+					(size 1.27 1.27)
+				)
+				(justify right)
+			)
+		)
+		(property "Footprint" "Resistor_SMD:R_0603_1608Metric_Pad0.98x0.95mm_HandSolder"
+			(at 91.948 43.18 90)
 			(effects
 				(font
@@
 		)
 		(property "Datasheet" "~"
-			(at 71.12 40.64 0)
-			(effects
-				(font
-					(size 1.27 1.27)
-				)
-				(hide yes)
-			)
-		)
-		(property "Description" "Generic connector, single row, 01x01, script generated"
-			(at 71.12 40.64 0)
+			(at 90.17 43.18 0)
+			(effects
+				(font
+					(size 1.27 1.27)
+				)
+				(hide yes)
+			)
+		)
+		(property "Description" "Resistor"
+			(at 90.17 43.18 0)
 			(effects
 				(font
@@
 		(pin "1"
 		)
+		(pin "2"
+		)
 		(instances
-			(project ""
+			(project "onyks-iot-esp32-storage-rfid"
 				(path "/d3620cad-99d5-4267-a144-49d6f9957c6b/de20a575-b588-4674-a6be-01e8d6418ae5"
-					(reference "J6")
+					(reference "R4")
 					(unit 1)
 				)
