File: pcb/onyks-iot-esp32-storage-rfid/onyks-iot-esp32-storage-rfid.kicad_pcb (KiCad board)
At the start: 4 copper layers, 46.8 x 48 mm, 25 parts, among them J1 Conn_01x02_Pin, J2 Conn_01x06_Pin, J3 Conn_02x05_Top_Bottom, J4 Conn_01x04_Pin, Q1 SS8050, Q2 SS8050, SW3 SW_Push, SW4 SW_Push, U1 ESP32-WROOM-32D, U2 TLV75733PDBV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

Commit message: male zmiany PCB
poprawiono niezmienione przelotki i usunieto powierzchnie masy pod U3
Routing:
- net VDD33: track 92.4 -> 86.1 mm
- net GND: vias 99 -> 97
Changed lines of the file:
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@@
 		(tags "resistor handsolder")
 		(property "Reference" "R2"
-			(at 0.1125 -1.6 0)
+			(at -2.679 -0.155 0)
 			(layer "F.SilkS")
 			(effects
@@
 			(keep_text_aligned yes)
 		)
-		(gr_text "48.00 mm"
+		(gr_text "48,00 mm"
 			(at 121.65 115.8 90)
 			(layer "Dwgs.User")
@@
 			(keep_text_aligned yes)
 		)
-		(gr_text "3.20 mm"
+		(gr_text "3,20 mm"
 			(at 130.8 86.25 0)
 			(layer "Dwgs.User")
@@
 			(keep_text_aligned yes)
 		)
-		(gr_text "46.80 mm"
+		(gr_text "46,80 mm"
 			(at 151.2 143.85 0)
 			(layer "Dwgs.User")
@@
 	)
 	(via
+		(at 132 104.2)
+		(size 0.6)
+		(drill 0.3)
+		(layers "F.Cu" "B.Cu")
+		(free yes)
+		(net 2)
+	)
+	(via
 		(at 142.621 104.14)
 		(size 0.6)
@@
 	)
 	(via
+		(at 129.4 103.2)
+		(size 0.6)
+		(drill 0.3)
+		(layers "F.Cu" "B.Cu")
+		(free yes)
+		(net 2)
+	)
+	(via
 		(at 151.257 119.634)
+		(size 0.6)
+		(drill 0.3)
+		(layers "F.Cu" "B.Cu")
+		(free yes)
+		(net 2)
+	)
+	(via
+		(at 129.4 98.8)
 		(size 0.6)
 		(drill 0.3)
@@
 	)
 	(via
-		(at 136.906 101.6)
-		(size 0.6)
-		(drill 0.3)
-		(layers "F.Cu" "B.Cu")
-		(free yes)
-		(net 2)
-	)
-	(via
 		(at 146.304 122.047)
 		(size 0.6)
@@
 	)
 	(via
-		(at 138.811 101.6)
-		(size 0.6)
-		(drill 0.3)
-		(layers "F.Cu" "B.Cu")
-		(free yes)
-		(net 2)
-	)
-	(via
 		(at 143.764 102.616)
 		(size 0.6)
@@
 	)
 	(via
-		(at 132.6 98)
-		(size 0.5)
-		(drill 0.3)
-		(layers "F.Cu" "B.Cu")
-		(free yes)
-		(tenting front back)
+		(at 132.2 97.6)
+		(size 0.6)
+		(drill 0.3)
+		(layers "F.Cu" "B.Cu")
+		(free yes)
 		(net 2)
 	)
@@
 	(via
 		(at 165.989 127)
-		(size 0.6)
-		(drill 0.3)
-		(layers "F.Cu" "B.Cu")
-		(free yes)
-		(net 2)
-	)
-	(via
-		(at 137.033 97.663)
 		(size 0.6)
 		(drill 0.3)
@@
 	)
 	(via
-		(at 166.243 102.87)
-		(size 0.5)
-		(drill 0.3)
-		(layers "F.Cu" "B.Cu")
-		(free yes)
-		(tenting front back)
-		(net 2)
-	)
-	(via
 		(at 163.195 92.71)
 		(size 0.5)
@@
 	)
 	(via
-		(at 129.413 103.378)
-		(size 0.6)
-		(drill 0.3)
-		(layers "F.Cu" "B.Cu")
-		(free yes)
-		(net 2)
-	)
-	(via
 		(at 129.413 125.73)
 		(size 0.6)
@@
 	)
 	(segment
-		(start 134.7 99.6)
-		(end 141 99.6)
-		(width 0.4)
-		(layer "F.Cu")
-		(net 3)
-	)
-	(segment
 		(start 164.4 103.2)
 		(end 164.4 100.8)
@@
 	(via
 		(at 162 117.6)
-		(size 0.5)
+		(size 0.6)
 		(drill 0.3)
 		(layers "F.Cu" "B.Cu")
@@
 	)
 	(zone
+		(net 0)
+		(net_name "")
+		(layer "F.Cu")
+		(hatch edge 0.5)
+		(connect_pads
+			(clearance 0)
+		)
+		(min_thickness 0.25)
+		(filled_areas_thickness no)
+		(keepout
+			(tracks not_allowed)
+			(vias not_allowed)
+			(pads allowed)
+			(copperpour not_allowed)
+			(footprints allowed)
+		)
+		(placement
+			(enabled no)
+			(sheetname "/ESP32/")
+		)
+		(fill
+			(thermal_gap 0.5)
+			(thermal_bridge_width 0.5)
+		)
+		(polygon
+			(pts
+				(xy 139.6 101.2) (xy 135.6 101.2) (xy 135.6 97.8) (xy 139.6 97.8)
+			)
+		)
+	)
+	(zone

Commit message: -
Routing:
- net VDD33: track 86.1 -> 92.4 mm
Changed lines of the file:
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@@
+	)
+	(segment
+		(start 134.7 99.6)
+		(end 141 99.6)
+		(width 0.4)
+		(layer "F.Cu")
+		(net 3)
 	)
 	(segment
@@
 		(filled_areas_thickness no)
 		(keepout
-			(tracks not_allowed)
+			(tracks allowed)
 			(vias not_allowed)
 			(pads allowed)
